File: hardware/controls-carier-board/controls-carier-board.kicad_sch (KiCad schematic)
At the start: 1 part, among them U1 BMM150

Commit message: fab version
Parts:
- removed U1: BMM150, Package_CSP:WLCSP-12_1.56x1.56mm_P0.4mm, symbol Sensor_Magnetic:BMM150
- added C1, C7: 10n, Capacitor_SMD:C_0603_1608Metric, symbol Device:C
- added C10, C11, C3, C4, C5, C6, C9: 0u1, Capacitor_SMD:C_0603_1608Metric, symbol Device:C
- added C14: 1u, Capacitor_SMD:C_0603_1608Metric, symbol Device:C
- added C15: 470p, Capacitor_SMD:C_0603_1608Metric, symbol Device:C
- added C16: 2u2, Capacitor_Tantalum_SMD:CP_EIA-3216-18_Kemet-A_Pad1.58x1.35mm_HandSolder, symbol Device:C_Polarized
- added C2, C8: 2u2, Capacitor_SMD:C_0603_1608Metric, symbol Device:C
- added D1: BAT760, Diode_SMD:D_SOD-323, symbol Diode:BAT760
- added D2, D3: LED, LED_SMD:LED_0603_1608Metric, symbol Device:LED
- added H1, H2, H3, H4: MountingHole_Pad, MountingHole:MountingHole_2.7mm_M2.5_Pad_Via, symbol Mechanical:MountingHole_Pad
- added J1, J2: DF40HC_4.0_-60DS-0.4V_51_, whose_lib:DF40HC4060DS04V51, symbol whose_lib:DF40HC_4.0_-60DS-0.4V_51_
- added R1, R10, R11, R12, R13, R14, R15, R16, R17, R18, R19, R2, R20, R21, R22, R23, R24, R3, R31, R32, R4, R5, R6, R9: 22, Resistor_SMD:R_0603_1608Metric, symbol Device:R
- added R33, R34: 330, Resistor_SMD:R_0603_1608Metric, symbol Device:R
- added R7, R8: 10k, Resistor_SMD:R_0603_1608Metric, symbol Device:R
- added SW1: SW_DIP_x02, whose_lib:218-2LPSTRF, symbol Switch:SW_DIP_x02
- added TP1, TP10, TP11, TP12, TP13, TP14, TP15, TP16, TP17, TP18, TP19, TP2, TP20, TP3, TP4, TP5, TP6, TP7, TP8, TP9: TestPoint, TestPoint:TestPoint_Keystone_5000-5004_Miniature, symbol Connector:TestPoint
- added U1: ICM-40609-D, whose_lib:ICM_LGA-24_3x3mm-P0.4mm, symbol whose_lib:ICM-40609-D
- added U2: BNO085X, Package_LGA:LGA-28_5.2x3.8mm_P0.5mm, symbol whose_lib:BNO085X
- added U3: ICM-42688-P, whose_lib:ICM_LGA-14_3x2.5mm_P0.5mm, symbol whose_lib:ICM-42688-P
- added U4: BMP390, whose_lib:Bosch_LGA-10_2x2mm_P0.50mm, symbol whose_lib:BMP390
- added U6: MIC5219-3.3YM5, Package_TO_SOT_SMD:SOT-23-5, symbol Regulator_Linear:MIC5219-3.3YM5
Connections:
- new net: C14.1, D1.1 (K), D2.2 (A), U6.1 (IN)
- new net: R9.1, TP1.1, U1.22 (nCS)
- new net: C15.1, U6.4 (BP)
- new net: R31.1, U3.9 (INT2/FSYNC/CLKIN)
- new net: R3.2, TP13.1, U2.19 (H_SCL/SCK/RX)
- new net: R13.1, U1.12 (INT1/INT)
- new net: R14.1, U1.19 (INT2/FSYNC)
- new net: R10.1, TP2.1, U1.23 (SCL/SCK)
- new net: R11.1, U1.24 (SDA/SDI/SDIO)
- new net: R12.1, U1.9 (AD0/SD0)
- new net: R21.1, TP16.1, U4.4 (SDI)
- new net: R23.1, TP18.1, U4.6 (CSB)
- new net: D3.1 (K), R34.2
- new net: R4.2, U2.14 (H_INTN)
- new net: D2.1 (K), R33.2
- new net: R2.2, TP12.1, U2.20 (H_SDA/MISO/TX)
- new net: R20.1, TP15.1, U4.2 (SCK)
- new net: R15.1, U2.11 (NRST)
- new net: R1.2, TP11.1, U2.17 (H_SA0/MOSI)
- new net: R6.2, TP14.1, U2.18 (H_CSN)
- new net: R5.2, U2.6 (PS0/WAKE)
- new net: R22.1, TP17.1, U4.5 (SDO)
- new net: R17.1, TP9.1, U3.1 (AP_SDO/AP_AD0)
- new net: R19.1, TP7.1, U3.12 (AP_CS)
- new net: R18.1, TP8.1, U3.13 (AP_SCL/AP_SCK)
- new net: R16.1, TP10.1, U3.14 (AP_SDA/AP_SDIO/AP_SDI)
- new net: R32.1, U3.4 (INT1/INT)
- new net: R24.1, U4.7 (INT)
- new net +3.3V: C1.1, C10.1, C11.1, C16.1, C2.1, C3.1, C4.1, C5.1, C6.1, C7.1, C8.1, C9.1, D3.2 (A), R7.2, R8.2, TP6.1, U1.13 (VDD), U1.8 (VDDIO), U2.10 (CLKSEL0), U2.28 (VDDIO), U2.3 (VDD), U2.9 (CAP), U3.5 (VDDIO), U3.8 (VDD), U4.1 (VDDIO), U4.10 (VDD), U6.5 (OUT)
- new net +5V: D1.2 (A), J1.51, J1.53, J1.55, J1.57, J1.59, J2.51, J2.53, J2.55, J2.57, J2.59, TP5.1
- new net 3V3_EN: J1.39, U6.3 (EN)
- new net BMP_CS: J2.31, R23.2
- new net BMP_INT: J2.29, R24.2
- new net BMP_SCK: J2.33, R20.2
- new net BMP_SDI: J2.37, R21.2
- new net BMP_SDO: J2.35, R22.2
- new net BN_BOOTN: R7.1, SW1.1, U2.4 (BOOTN)
- new net BN_CS: J1.2, R6.1
- new net BN_INT: J1.12, R4.1
- new net BN_MISO: J1.8, R2.1
- new net BN_MOSI: J1.10, R1.1
- new net BN_NRST: J1.14, R15.2
- new net BN_PS0: J1.18, R5.1
- new net BN_PS1: R8.1, SW1.2, U2.5 (PS1)
- new net BN_SCK: J1.4, R3.1
- new net GND: C1.2, C10.2, C11.2, C14.2, C15.2, C16.2, C2.2, C3.2, C4.2, C5.2, C6.2, C7.2, C8.2, C9.2, H1.1, H2.1, H3.1, H4.1, J1.46, J1.48, J1.50, J1.52, J1.54, J1.56, J1.58, J1.60, J2.46, J2.48, J2.50, J2.52, J2.54, J2.56, J2.58, J2.60, R33.1, R34.1, SW1.3, SW1.4, TP19.1, TP20.1, U1.11 (RESV), U1.18 (GND), U1.20 (RESV), U2.2 (GND), U2.25 (GNDIO), U2.26 (XOUT32/CLKSEL1), U3.10 (RESV), U3.11 (RESV), U3.2 (RESV), U3.3 (RESV), U3.6 (GND), U3.7 (RESV), U4.3 (VSS), U4.8 (VSS), U4.9 (VSS), U6.2 (GND)
- new net ICM40609D_CS: J2.4, R9.2
- new net ICM40609D_INT1: J2.5, R13.2
- new net ICM40609D_INT2: J2.1, R14.2
- new net ICM40609D_SCK: J2.6, R10.2
- new net ICM40609D_SDI: J2.10, R11.2, TP4.1
- new net ICM40609D_SDO: J2.8, R12.2, TP3.1
- new net ICM42688P_CS: J1.1, R19.2
- new net ICM42688P_INT1: J1.29, R32.2
- new net ICM42688P_INT2: J1.31, R31.2
- new net ICM42688P_SCK: J1.3, R18.2
- new net ICM42688P_SDI: J1.27, R16.2
- new net ICM42688P_SDO: J1.25, R17.2
- no-connect marks 0 -> 72
Other:
- note added: "5V to 3V3"
- note added: "BMP390"
- note added: "BNO085X"
- note added: "CONN A"
- note added: "CONN B"
- note added: "Connector"
- note added: "ICM40609D"
- note added: "ICM42688P"
- note added: "Mounting Hole"
- note removed: "BNO085 : LGA-28pin 0.5mm pitch"
- title: (none) -> IMU Sensor Module
